File: Arduino_8FSR.sch (EAGLE design)
At the start: 17 parts, among them IC1 7805TV, IC2 UA741P, U1 HCF4051BEY, X2 TSW-117-08-G-S, X3 TSW-117-08-G-S, X4 057-006-1, X5 057-010-1

Commit message: Final Version
Parts:
- removed SV1: (no value), con-lsta:FE06-1
- removed X4: 057-006-1, con-panduit:057-006-1
- removed X5: 057-010-1, con-panduit:057-010-1
- added X6: 057-016-1, con-panduit:057-016-1
Connections:
- removed net AD0: U$2.D4*, X3-9.1, X4-5.S
- removed net EN: SV1.1, U$2.D7, X3-6.1
- removed net RXTX: SV1.5, U$2.D1/TX, X3-15.1
- removed net STATE: SV1.6, U$2.D6*, X3-7.1
- removed net TXRX: SV1.4, U$2.D0/RX, X3-14.1
- new net N$10: U$2.D1/TX, X3-15.1
- new net N$4: U$2.D5*, X3-8.1
- new net N$7: U$2.D6*, X3-7.1
- new net N$8: U$2.D7, X3-6.1
- new net N$9: U$2.D4*, X3-9.1
- new net NC: X6-15.S
- net GND: now also X6-12.S; no longer SV1.3, X4-2.S
- net INT: now also U$2.D0/RX, X3-14.1, X6-16.S; no longer U$2.D5*, X3-8.1, X4-6.S
- net IP1: now also X6-3.S; no longer X5-3.S
- net IP2: now also X6-4.S; no longer X5-4.S
- net IP3: now also X6-5.S; no longer X5-5.S
- net IP4: now also X6-6.S; no longer X5-6.S
- net IP5: now also X6-7.S; no longer X5-7.S
- net IP6: now also X6-8.S; no longer X5-8.S
- net IP7: now also X6-9.S; no longer X5-9.S
- net IP8: now also X6-10.S; no longer X5-10.S
- net SCL: now also X6-13.S; no longer X4-3.S
- net SDA: now also X6-14.S; no longer X4-4.S
- net VCC_5V: now also X6-1.S, X6-11.S, X6-2.S; no longer SV1.2, X4-1.S, X5-1.S, X5-2.S

Commit message: Final update V1
Parts:
- added R2, R3: (no value), rcl:R-US_0204/7
Connections:
- net SCL: now also R3.1
- net SDA: now also R2.1
- net VCC_5V: now also R2.2, R3.2
Other:
- moved on the sheet: X3-10, X3-11
Changed lines of the file:
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@@
 <part name="H4" library="holes" library_urn="urn:adsk.eagle:library:237" deviceset="MOUNT-HOLE" device="3.0" package3d_urn="urn:adsk.eagle:package:14277/1"/>
 <part name="X6" library="con-panduit" library_urn="urn:adsk.eagle:library:169" deviceset="057-016-" device="1" package3d_urn="urn:adsk.eagle:package:9196/1"/>
+<part name="R2" library="rcl" library_urn="urn:adsk.eagle:library:334" deviceset="R-US_" device="0204/7" package3d_urn="urn:adsk.eagle:package:23498/2"/>
+<part name="R3" library="rcl" library_urn="urn:adsk.eagle:library:334" deviceset="R-US_" device="0204/7" package3d_urn="urn:adsk.eagle:package:23498/2"/>
 </parts>
 <sheets>
@@
 <attribute name="NAME" x="74.93" y="120.142" size="1.524" layer="95" rot="R180"/>
 </instance>
-<instance part="X3" gate="-10" x="77.47" y="121.92" smashed="yes" rot="R180">
-<attribute name="NAME" x="74.93" y="122.682" size="1.524" layer="95" rot="R180"/>
-</instance>
-<instance part="X3" gate="-11" x="77.47" y="124.46" smashed="yes" rot="R180">
-<attribute name="NAME" x="74.93" y="125.222" size="1.524" layer="95" rot="R180"/>
+<instance part="X3" gate="-10" x="39.37" y="121.92" smashed="yes" rot="R180">
+<attribute name="NAME" x="36.83" y="122.682" size="1.524" layer="95" rot="R180"/>
+</instance>
+<instance part="X3" gate="-11" x="59.69" y="124.46" smashed="yes" rot="R180">
+<attribute name="NAME" x="57.15" y="125.222" size="1.524" layer="95" rot="R180"/>
 </instance>
 <instance part="X3" gate="-12" x="77.47" y="127" smashed="yes" rot="R180">
@@
 <instance part="X6" gate="-16" x="132.08" y="45.72" smashed="yes">
 <attribute name="NAME" x="133.096" y="44.958" size="1.524" layer="95"/>
+</instance>
+<instance part="R2" gate="G$1" x="63.5" y="129.54" smashed="yes" rot="R90">
+<attribute name="NAME" x="62.0014" y="125.73" size="1.778" layer="95" rot="R90"/>
+<attribute name="VALUE" x="66.802" y="125.73" size="1.778" layer="96" rot="R90"/>
+</instance>
+<instance part="R3" gate="G$1" x="43.18" y="127" smashed="yes" rot="R90">
+<attribute name="NAME" x="41.6814" y="123.19" size="1.778" layer="95" rot="R90"/>
+<attribute name="VALUE" x="46.482" y="123.19" size="1.778" layer="96" rot="R90"/>
 </instance>
 </instances>
@@
 <pinref part="X6" gate="-11" pin="S"/>
 </segment>
+<segment>
+<pinref part="R3" gate="G$1" pin="2"/>
+<wire x1="43.18" y1="132.08" x2="43.18" y2="134.62" width="0.1524" layer="91"/>
+<pinref part="R2" gate="G$1" pin="2"/>
+<wire x1="43.18" y1="134.62" x2="53.34" y2="134.62" width="0.1524" layer="91"/>
+<wire x1="53.34" y1="134.62" x2="63.5" y2="134.62" width="0.1524" layer="91"/>
+<wire x1="53.34" y1="134.62" x2="53.34" y2="139.7" width="0.1524" layer="91"/>
+<wire x1="53.34" y1="139.7" x2="63.5" y2="139.7" width="0.1524" layer="91"/>
+<junction x="53.34" y="134.62"/>
+<label x="55.88" y="139.7" size="1.778" layer="95"/>
+</segment>
 </net>
 <net name="N$1" class="0">
@@
 <pinref part="X3" gate="-10" pin="1"/>
 <pinref part="U$2" gate="G$1" pin="D3/SCL"/>
-<wire x1="80.01" y1="121.92" x2="88.9" y2="121.92" width="0.1524" layer="91"/>
+<wire x1="41.91" y1="121.92" x2="43.18" y2="121.92" width="0.1524" layer="91"/>
 <label x="81.28" y="121.92" size="1.778" layer="95"/>
+<pinref part="R3" gate="G$1" pin="1"/>
+<wire x1="43.18" y1="121.92" x2="88.9" y2="121.92" width="0.1524" layer="91"/>
+<junction x="43.18" y="121.92"/>
 </segment>
 </net>
@@
 <pinref part="X3" gate="-11" pin="1"/>
 <pinref part="U$2" gate="G$1" pin="D2/SDA"/>
-<wire x1="80.01" y1="124.46" x2="88.9" y2="124.46" width="0.1524" layer="91"/>
+<wire x1="62.23" y1="124.46" x2="63.5" y2="124.46" width="0.1524" layer="91"/>
 <label x="81.28" y="124.46" size="1.778" layer="95"/>
-</segment>
-</net>
+<pinref part="R2" gate="G$1" pin="1"/>
+<wire x1="63.5" y1="124.46" x2="88.9" y2="124.46" width="0.1524" layer="91"/>
+<junction x="63.5" y="124.46"/>
+</segment>
+</net>
